File: Hardware/Plugin Arduino Shield/v2.0/PuM_Arduino_Shield_v2.brd (EAGLE design)
At the start: 73.9 x 53.3 mm, 47 parts, among them P2 RF_SMA, P5 USB-MICROB, U1 LMZ12002TZ-ADJ, U2 TERMINUS_X910CF, U3 SN74LVC2T45DCT, U4 SN74LVC2T45DCT

Commit message: Updated board design and library
Parts:
- JP3: device SparkFun-Retired:SJ_2S -> SparkFun-Retired:SJ_2S-NO
- JP6: device SparkFun-Retired:SJ_2S-NO -> SparkFun-Retired:SJ_2S
Other:
- board text added: "P1"
- board text added: "P3"
- board text added: "P4"
- board text added: "P6"
- board text added: "P7"
- board text added: "P8"
- board text added: "P9"
- board text removed: "LAYER-STACK"
Changed lines of the file:
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@@
 <layer number="27" name="tValues" color="7" fill="1" visible="no" active="yes"/>
 <layer number="28" name="bValues" color="7" fill="1" visible="no" active="yes"/>
-<layer number="29" name="tStop" color="7" fill="3" visible="no" active="yes"/>
+<layer number="29" name="tStop" color="7" fill="3" visible="yes" active="yes"/>
 <layer number="30" name="bStop" color="7" fill="6" visible="no" active="yes"/>
 <layer number="31" name="tCream" color="7" fill="4" visible="no" active="yes"/>
@@
 <layer number="131" name="tAdjust" color="7" fill="1" visible="no" active="yes"/>
 <layer number="132" name="bAdjust" color="7" fill="1" visible="no" active="yes"/>
-<layer number="144" name="DrillLegend" color="7" fill="1" visible="no" active="yes"/>
+<layer number="144" name="DrillLegend" color="7" fill="1" visible="yes" active="yes"/>
 <layer number="145" name="DrillLegend_01-16" color="2" fill="9" visible="no" active="yes"/>
 <layer number="146" name="DrillLegend_01-20" color="3" fill="9" visible="no" active="yes"/>
@@
 <wire x1="48.4" y1="32.2" x2="49.2" y2="32.2" width="0.2032" layer="21"/>
 <wire x1="49.2" y1="32.2" x2="49.2" y2="33.2" width="0.2032" layer="21"/>
-<text x="-19.685" y="-3.81" size="1.778" layer="144">LAYER-STACK</text>
 <text x="-9.906" y="-6.7437" size="1.778" layer="145">01-16</text>
 <wire x1="54.483" y1="29.718" x2="54.483" y2="28.702" width="0.1016" layer="145"/>
@@
 <wire x1="66.548" y1="8.5725" x2="66.548" y2="7.5565" width="0.1016" layer="146"/>
 <wire x1="66.548" y1="7.5565" x2="66.04" y2="8.0645" width="0.1016" layer="146"/>
+<text x="71.1" y="40.2" size="0.8128" layer="25" font="vector">P1</text>
+<text x="27.2" y="4.4" size="0.8128" layer="25" font="vector">P3</text>
+<text x="45" y="52.6" size="0.8128" layer="25" font="vector">P4</text>
+<text x="48.6" y="3.4" size="0.8128" layer="25" font="vector">P6</text>
+<text x="18.3" y="52.6" size="0.8128" layer="25" font="vector">P7</text>
+<text x="61" y="38.6" size="0.8128" layer="25" font="vector">P8</text>
+<text x="62.1" y="14.3" size="0.8128" layer="25" font="vector">P9</text>
 </plain>
 <attributes>
@@
 </element>
 <element name="D1" library="SparkFun-LED" package="LED-0603" value="" x="15.3797" y="2.1844" smashed="yes" rot="R270">
-<attribute name="NAME" x="17.8054" y="1.6256" size="0.8128" layer="25"/>
+<attribute name="NAME" x="17.8054" y="1.6256" size="0.8128" layer="25" font="vector"/>
 <attribute name="VALUE" x="14.3637" y="1.1049" size="0.4064" layer="27"/>
 </element>
@@
 <attribute name="VALUE" x="49.657" y="47.4535" size="0.4064" layer="27" rot="R270"/>
 </element>
-<element name="JP6" library="SparkFun-Retired" package="SJ_2S-NO" value="" x="51.308" y="7.3025" smashed="yes" rot="R90">
+<element name="JP6" library="SparkFun-Retired" package="SJ_2S" value="" x="51.308" y="7.3025" smashed="yes" rot="R90">
 <attribute name="NAME" x="50.4" y="9.2075" size="0.8128" layer="25"/>
 <attribute name="VALUE" x="52.959" y="6.3945" size="0.4064" layer="27" rot="R90"/>
@@
 <attribute name="VALUE" x="67.31" y="43.8785" size="1.778" layer="27" rot="R270"/>
 </element>
-<element name="JP3" library="SparkFun-Retired" package="SJ_2S" value="" x="7.366" y="52.2605" smashed="yes">
+<element name="JP3" library="SparkFun-Retired" package="SJ_2S-NO" value="" x="7.366" y="52.2605" smashed="yes">
 <attribute name="NAME" x="6.5432" y="50.1015" size="0.8128" layer="25"/>
 <attribute name="VALUE" x="6.4162" y="50.6095" size="0.4064" layer="27"/>
@@
 <contactref element="JP5" pad="1"/>
 <contactref element="ARD1" pad="D6"/>
-<wire x1="48.768" y1="46.9574" x2="48.768" y2="51.2445" width="0.2032" layer="1"/>
+<wire x1="48.768" y1="46.9447" x2="48.768" y2="51.2445" width="0.2032" layer="1"/>
 </signal>
 <signal name="SW_TXD">
@@
 <wire x1="45.085" y1="12.8905" x2="50.223" y2="7.7525" width="0.2032" layer="1"/>
 <wire x1="50.223" y1="7.7525" x2="51.308" y2="7.7525" width="0.2032" layer="1"/>
+<wire x1="51.308" y1="7.7525" x2="51.308" y2="7.7017" width="0.2032" layer="1"/>
 </signal>
 <signal name="MDM_ENABLE">
@@
 <contactref element="JP7" pad="2"/>
 <contactref element="P3" pad="3"/>
-<wire x1="27.305" y1="12.8905" x2="27.305" y2="16.4774" width="0.2032" layer="1"/>
-<wire x1="27.305" y1="16.4774" x2="27.4011" y2="16.5735" width="0.2032" layer="1"/>
+<wire x1="27.305" y1="16.4774" x2="27.4138" y2="16.5735" width="0.2032" layer="1"/>
 <wire x1="8.509" y1="4.2545" x2="7.239" y2="2.9845" width="0.2032" layer="16"/>
+<wire x1="27.305" y1="12.8905" x2="27.305" y2="16.5735" width="0.2032" layer="1"/>
+<wire x1="27.305" y1="16.5735" x2="27.4138" y2="16.5735" width="0.2032" layer="1"/>
 </signal>
 <signal name="VBUS">
@@
 <wire x1="11.43" y1="50.8635" x2="10.48" y2="51.8135" width="0.2032" layer="1"/>
 <wire x1="10.48" y1="51.8135" x2="10.414" y2="51.8135" width="0.2032" layer="1"/>
-<wire x1="7.7779" y1="52.2605" x2="9.967" y2="52.2605" width="0.2032" layer="1"/>
+<wire x1="7.816" y1="52.2605" x2="9.967" y2="52.2605" width="0.2032" layer="1"/>
 <wire x1="9.967" y1="52.2605" x2="10.414" y2="51.8135" width="0.2032" layer="1"/>
 <wire x1="11.43" y1="48.895" x2="12.8905" y2="47.4345" width="0.2032" layer="1"/>
@@
 <wire x1="52.6" y1="48.05" x2="52.6" y2="46.4" width="0.2032" layer="1"/>
 <wire x1="52.6" y1="46.4" x2="52.9" y2="46.1" width="0.2032" layer="1"/>
-<wire x1="52.9" y1="46.1" x2="53.8435" y2="46.1" width="0.2032" layer="1"/>
-<wire x1="53.8435" y1="46.1" x2="53.848" y2="46.1336" width="0.2032" layer="1"/>
+<wire x1="53.8435" y1="46.1" x2="53.848" y2="46.1463" width="0.2032" layer="1"/>
+<wire x1="52.9" y1="46.1" x2="53.848" y2="46.1" width="0.2032" layer="1"/>
+<wire x1="53.848" y1="46.1" x2="53.848" y2="46.1463" width="0.2032" layer="1"/>
 </signal>
 <signal name="MDM_USB_D+">
@@
 <wire x1="42.55" y1="44.4" x2="44.2" y2="46.05" width="0.2032" layer="16"/>
 <wire x1="44.2" y1="46.05" x2="46.3" y2="46.05" width="0.2032" layer="16"/>
-<wire x1="48.768" y1="46.1336" x2="46.3455" y2="46.0955" width="0.2032" layer="1"/>
-<wire x1="46.3455" y1="46.0955" x2="46.3" y2="46.05" width="0.2032" layer="1"/>
+<wire x1="46.3" y1="46.1717" x2="46.3" y2="46.05" width="0.2032" layer="1"/>
+<wire x1="48.768" y1="46.1463" x2="46.3" y2="46.1463" width="0.2032" layer="1"/>
+<wire x1="46.3" y1="46.1463" x2="46.3" y2="46.05" width="0.2032" layer="1"/>
 </signal>
 <signal name="DVI_CLK">
@@
 <contactref element="JP4" pad="1"/>
 <contactref element="ARD1" pad="D5"/>
-<wire x1="51.308" y1="46.9574" x2="51.308" y2="51.2445" width="0.2032" layer="1"/>
+<wire x1="51.308" y1="46.9447" x2="51.308" y2="51.2445" width="0.2032" layer="1"/>
 </signal>
 <signal name="N$7">
@@
 <wire x1="50" y1="48.05" x2="50" y2="46.5" width="0.2032" layer="1"/>
 <wire x1="50" y1="46.5" x2="50.4" y2="46.1" width="0.2032" layer="1"/>
-<wire x1="50.4" y1="46.1" x2="51.3035" y2="46.1" width="0.2032" layer="1"/>
-<wire x1="51.3035" y1="46.1" x2="51.308" y2="46.1336" width="0.2032" layer="1"/>
+<wire x1="51.3035" y1="46.1" x2="51.308" y2="46.1463" width="0.2032" layer="1"/>
 <wire x1="45.1" y1="39.25" x2="45.1" y2="43.15" width="0.2032" layer="16"/>
 <wire x1="45.1" y1="43.15" x2="50" y2="48.05" width="0.2032" layer="16"/>
+<wire x1="50.4" y1="46.1" x2="51.308" y2="46.1" width="0.2032" layer="1"/>
+<wire x1="51.308" y1="46.1" x2="51.308" y2="46.1463" width="0.2032" layer="1"/>
 </signal>
 <signal name="ARD_A0">
 <contactref element="JP6" pad="1"/>
 <contactref element="ARD1" pad="A0"/>
-<wire x1="51.308" y1="2.9845" x2="51.308" y2="6.8525" width="0.2032" layer="1"/>
+<wire x1="51.308" y1="2.9845" x2="51.308" y2="6.9033" width="0.2032" layer="1"/>
 </signal>
 <signal name="ARD_D4">
 <contactref element="JP8" pad="1"/>
 <contactref element="ARD1" pad="D4"/>
-<wire x1="53.848" y1="46.9574" x2="53.848" y2="51.2445" width="0.2032" layer="1"/>
+<wire x1="53.848" y1="46.9447" x2="53.848" y2="51.2445" width="0.2032" layer="1"/>
 </signal>
 <signal name="MDM_SCL">
