File: Hardware/Plugin Arduino Shield/v2.0/PuM_Arduino_Shield_v2.sch (EAGLE design)
At the start: 45 parts, among them P2 RF_SMA, P5 USB-MICROB, U1 LMZ12002TZ-ADJ, U2 TERMINUS_X910CF, U3 SN74LVC2T45DCT, U4 SN74LVC2T45DCT

Commit message: Updated board design and library
Parts:
- JP3: device SparkFun-Retired:JUMPER-2SMD-NC -> SparkFun-Retired:JUMPER-2SMD-NO
- JP6: device SparkFun-Retired:JUMPER-2SMD-NO -> SparkFun-Retired:JUMPER-2SMD-NC
Changed lines of the file:
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@@
 <setting verticaltext="up"/>
 </settings>
-<grid distance="0.05" unitdist="inch" unit="inch" style="lines" multiple="1" display="yes" altdistance="0.01" altunitdist="inch" altunit="inch"/>
+<grid distance="0.1" unitdist="inch" unit="inch" style="lines" multiple="1" display="no" altdistance="0.01" altunitdist="inch" altunit="inch"/>
 <layers>
 <layer number="1" name="Top" color="4" fill="1" visible="no" active="no"/>
@@
 <part name="GND6" library="supply1" deviceset="GND" device=""/>
 <part name="JP4" library="SparkFun-Retired" deviceset="JUMPER-2" device="SMD-NC"/>
-<part name="JP6" library="SparkFun-Retired" deviceset="JUMPER-2" device="SMD-NO"/>
+<part name="JP6" library="SparkFun-Retired" deviceset="JUMPER-2" device="SMD-NC"/>
 <part name="JP7" library="SparkFun-Retired" deviceset="JUMPER-2" device="SMD-NC"/>
 <part name="P1" library="Connector" deviceset="HEADER-2X3P" device="-2.54"/>
-<part name="JP3" library="SparkFun-Retired" deviceset="JUMPER-2" device="SMD-NC"/>
+<part name="JP3" library="SparkFun-Retired" deviceset="JUMPER-2" device="SMD-NO"/>
 <part name="JP8" library="SparkFun-Retired" deviceset="JUMPER-2" device="SMD-NC"/>
 <part name="P2" library="Janus-IC" deviceset="RF_SMA" device=""/>
